Commit message: v1 robot integration

File: v1_urdf/robot.urdf (robot description, URDF)
Before this commit: robot humanoid_robot, 25 links, 24 joints
Links:
- link bearing: geometry collision mesh filename=package://my_robot_description/v1_meshes/merged/bearing_col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; visual mesh filename=package://my_robot_description/v1_meshes/merged/bearing_vis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
- link bicep: geometry collision mesh filename=package://my_robot_description/v1_meshes/merged/bicep_colli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; visual mesh filename=package://my_robot_description/v1_meshes/merged/bicep_visua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
- link camera_enclosure: geometry collision mesh filename=package://my_robot_description/v1_meshes/merged/camera_encl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; visual mesh filename=package://my_robot_description/v1_meshes/merged/camera_encl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
- link foot: geometry collision mesh filename=package://my_robot_description/v1_meshes/merged/foot_collis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; visual mesh filename=package://my_robot_description/v1_meshes/merged/foot_visual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
- link foot_2: geometry collision mesh filename=package://my_robot_description/v1_meshes/merged/foot_collis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; visual mesh filename=package://my_robot_description/v1_meshes/merged/foot_visual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
- link forearm: geometry collision mesh filename=package://my_robot_description/v1_meshes/merged/forearm_col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; visual mesh filename=package://my_robot_description/v1_meshes/merged/forearm_vis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
- link knee_ankle_rotor_case: geometry collision mesh filename=package://my_robot_description/v1_meshes/merged/knee_ankle_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; visual mesh filename=package://my_robot_description/v1_meshes/merged/knee_ankle_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
- link knee_ankle_rotor_case_2: geometry collision mesh filename=package://my_robot_description/v1_meshes/merged/knee_ankle_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; visual mesh filename=package://my_robot_description/v1_meshes/merged/knee_ankle_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
- link knee_housing: geometry collision mesh filename=package://my_robot_description/v1_meshes/merged/knee_housin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; visual mesh filename=package://my_robot_description/v1_meshes/merged/knee_housin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
- link pitch_roll_housing: geometry collision mesh filename=package://my_robot_description/v1_meshes/merged/pitch_roll_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; visual mesh filename=package://my_robot_description/v1_meshes/merged/pitch_roll_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
- link shoulder_rightangle: geometry collision mesh filename=package://my_robot_description/v1_meshes/merged/shoulder_ri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; visual mesh filename=package://my_robot_description/v1_meshes/merged/shoulder_ri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
- link shoulder_rightangle_2: geometry collision mesh filename=package://my_robot_description/v1_meshes/merged/shoulder_ri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; visual mesh filename=package://my_robot_description/v1_meshes/merged/shoulder_ri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
- link sts3250: geometry collision mesh filename=package://my_robot_description/v1_meshes/merged/sts3250_col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; visual mesh filename=package://my_robot_description/v1_meshes/merged/sts3250_vis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
- link sts3250_2: geometry collision mesh filename=package://my_robot_description/v1_meshes/merged/knee_housin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; visual mesh filename=package://my_robot_description/v1_meshes/merged/knee_housin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
- link sts3250_3: geometry collision mesh filename=package://my_robot_description/v1_meshes/merged/sts3250_col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; visual mesh filename=package://my_robot_description/v1_meshes/merged/sts3250_vis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
- link sts3250_4: geometry collision mesh filename=package://my_robot_description/v1_meshes/merged/bicep_colli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; visual mesh filename=package://my_robot_description/v1_meshes/merged/bicep_visua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
- link sts3250_5: geometry collision mesh filename=package://my_robot_description/v1_meshes/merged/forearm_col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; visual mesh filename=package://my_robot_description/v1_meshes/merged/forearm_vis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
- link sts3250_6: geometry collision mesh filename=package://my_robot_description/v1_meshes/merged/sts3250_col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; visual mesh filename=package://my_robot_description/v1_meshes/merged/sts3250_vis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
- link torso: geometry collision mesh filename=package://my_robot_description/v1_meshes/merged/torso_colli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; visual mesh filename=package://my_robot_description/v1_meshes/merged/torso_visua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
- link yaw_adapter: geometry collision mesh filename=package://my_robot_description/v1_meshes/merged/yaw_adapter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; visual mesh filename=package://my_robot_description/v1_meshes/merged/yaw_adapter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
- link yaw_adapter_2: geometry collision mesh filename=package://my_robot_description/v1_meshes/merged/yaw_adapter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; visual mesh filename=package://my_robot_description/v1_meshes/merged/yaw_adapter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
Joints:
- joint left_foot_to_sole: origin xyz=0 0.03 -0.048 rpy=0 0 0 -> xyz=0 0.027 -0.0275 rpy=1.57079632679 1.57079632679 0
- joint right_foot_to_sole: origin xyz=0 0.03 -0.048 rpy=0 0 0 -> xyz=0 0.027 -0.0275 rpy=1.57079632679 1.57079632679 0
